File: electronics/Keyboard.sch (KiCad schematic (older format))
At the start: 4 parts, among them IC1 Teensy++2.0, J1 Input 5v, J1 Rows, J2 Columns

Commit message: COLS redraw to shorten wires
Connections:
- wire segments 57 -> 50
Changed lines of the file:
@@
 L Connector_Generic:Conn_01x02 J1
 U 1 1 5E771D4E
-P 3400 2200
-F 0 "J1" H 3318 1875 50  0001 C CNN
-F 1 "Input 5v" H 3318 1966 50  0000 C CNB
-F 2 "" H 3400 2200 50  0001 C CNN
-F 3 "~" H 3400 2200 50  0001 C CNN
-F 4 "GND" H 3150 2150 50  0000 C CNN "2"
-F 5 "Vcc" H 3150 2050 50  0000 C CNN "1"
-	1    3400 2200
+P 3050 2350
+F 0 "J1" H 2968 2025 50  0001 C CNN
+F 1 "Input 5v" H 2968 2116 50  0000 C CNB
+F 2 "" H 3050 2350 50  0001 C CNN
+F 3 "~" H 3050 2350 50  0001 C CNN
+F 4 "GND" H 2800 2300 50  0000 C CNN "2"
+F 5 "Vcc" H 2800 2200 50  0000 C CNN "1"
+	1    3050 2350
 	-1   0    0    1
 $EndComp
@@
 1
 Wire Wire Line
-	5900 2100 5900 2700
+	5900 2250 5900 2700
 Wire Wire Line
-	4650 2200 4650 2700
+	4650 2350 4650 2700
 $Comp
 L teensy:Teensy++2.0-teensy++20 IC1
@@
 $EndComp
 Wire Wire Line
-	3600 2200 4650 2200
+	3250 2350 4650 2350
 Wire Wire Line
-	3600 2100 5900 2100
+	3250 2250 5900 2250
 $Comp
 L Connector:Conn_01x06_Male J1
@@
 L Connector:Conn_01x20_Male J2
 U 1 1 5EF43085
-P 7250 3700
-F 0 "J2" H 7000 3750 50  0000 R CNN
-F 1 "Columns" H 7100 3650 50  0000 R CNN
-F 2 "" H 7250 3700 50  0001 C CNN
-F 3 "~" H 7250 3700 50  0001 C CNN
-	1    7250 3700
-	-1   0    0    -1
+P 3000 4500
+F 0 "J2" H 2750 4550 50  0000 R CNN
+F 1 "Columns" H 2850 4450 50  0000 R CNN
+F 2 "" H 3000 4500 50  0001 C CNN
+F 3 "~" H 3000 4500 50  0001 C CNN
+	1    3000 4500
+	1    0    0    -1
 $EndComp
 Wire Wire Line
-	5900 2800 7050 2800
+	4650 4500 3200 4500
 Wire Wire Line
-	5900 2900 7050 2900
+	4650 4400 3200 4400
 Wire Wire Line
-	5900 3000 7050 3000
+	3200 3600 4650 3600
 Wire Wire Line
-	5900 3100 7050 3100
+	3200 3700 4650 3700
 Wire Wire Line
-	5900 3200 7050 3200
+	3200 3800 4650 3800
 Wire Wire Line
-	5900 3300 7050 3300
+	3200 3900 4650 3900
 Wire Wire Line
-	5900 3400 7050 3400
+	3200 4000 4650 4000
 Wire Wire Line
-	5900 3500 7050 3500
+	3200 4100 4650 4100
 Wire Wire Line
-	5900 3600 7050 3600
+	3200 4200 4650 4200
 Wire Wire Line
-	5900 3900 6000 3900
+	3200 4300 4650 4300
 Wire Wire Line
-	6000 3900 6000 3700
+	4650 4600 3200 4600
 Wire Wire Line
-	6000 3700 7050 3700
+	5950 4750 5950 4600
 Wire Wire Line
-	5900 4000 6100 4000
+	5950 4600 5900 4600
 Wire Wire Line
-	6100 4000 6100 3800
+	3200 4800 6050 4800
 Wire Wire Line
-	6100 3800 7050 3800
+	6050 4800 6050 4500
 Wire Wire Line
-	5900 4100 6200 4100
+	6050 4500 5900 4500
 Wire Wire Line
-	6200 4100 6200 3900
+	4600 4750 5950 4750
 Wire Wire Line
-	6200 3900 7050 3900
+	4600 4700 4600 4750
 Wire Wire Line
-	5900 4200 6300 4200
+	3200 4700 4600 4700
 Wire Wire Line
-	6300 4200 6300 4000
+	3200 4900 6150 4900
 Wire Wire Line
-	6300 4000 7050 4000
+	6150 4900 6150 4400
 Wire Wire Line
-	5900 4300 6400 4300
+	6150 4400 5900 4400
 Wire Wire Line
-	6400 4300 6400 4100
+	5900 4300 6250 4300
 Wire Wire Line
-	6400 4100 7050 4100
+	6250 4300 6250 5000
 Wire Wire Line
-	5900 4400 6500 4400
+	6250 5000 3200 5000
 Wire Wire Line
-	6500 4400 6500 4200
+	3200 5100 6350 5100
 Wire Wire Line
-	6500 4200 7050 4200
+	6350 5100 6350 3600
 Wire Wire Line
-	5900 4500 6600 4500
+	6350 3600 5900 3600
 Wire Wire Line
-	6600 4500 6600 4300
+	5900 3500 6450 3500
 Wire Wire Line
-	6600 4300 7050 4300
+	6450 3500 6450 5200
 Wire Wire Line
-	5900 4600 6700 4600
+	6450 5200 3200 5200
 Wire Wire Line
-	6700 4600 6700 4400
+	3200 5300 6550 5300
 Wire Wire Line
-	6700 4400 7050 4400
+	6550 5300 6550 3000
 Wire Wire Line
-	4650 4600 4650 4800
+	6550 3000 5900 3000
 Wire Wire Line
-	4650 4800 6800 4800
+	5900 2900 6650 2900
 Wire Wire Line
-	6800 4800 6800 4500
+	6650 2900 6650 5400
 Wire Wire Line
-	6800 4500 7050 4500
+	6650 5400 3200 5400
 Wire Wire Line
-	4650 4500 4550 4500
+	3200 5500 6750 5500
 Wire Wire Line
-	4550 4500 4550 4900
+	6750 5500 6750 2800
 Wire Wire Line
-	4550 4900 6900 4900
-Wire Wire Line
-	6900 4900 6900 4600
-Wire Wire Line
-	6900 4600 7050 4600
-Wire Wire Line
-	4650 4400 4450 4400
-Wire Wire Line
-	4450 4400 4450 5000
-Wire Wire Line
-	4450 5000 7000 5000
-Wire Wire Line
-	7000 5000 7000 4700
-Wire Wire Line
-	7000 4700 7050 4700
+	6750 2800 5900 2800
 $EndSCHEMATC

Commit message: keyboard schematics updated
Connections:
- wire segments 50 -> 88
Other:
- note added: "Internal\nLED"
Changed lines of the file:
@@
 L Connector_Generic:Conn_01x02 J1
 U 1 1 5E771D4E
-P 3050 2350
-F 0 "J1" H 2968 2025 50  0001 C CNN
-F 1 "Input 5v" H 2968 2116 50  0000 C CNB
-F 2 "" H 3050 2350 50  0001 C CNN
-F 3 "~" H 3050 2350 50  0001 C CNN
-F 4 "GND" H 2800 2300 50  0000 C CNN "2"
-F 5 "Vcc" H 2800 2200 50  0000 C CNN "1"
-	1    3050 2350
+P 3600 1750
+F 0 "J1" H 3518 1425 50  0001 C CNN
+F 1 "Input 5v" H 3518 1516 50  0000 C CNB
+F 2 "" H 3600 1750 50  0001 C CNN
+F 3 "~" H 3600 1750 50  0001 C CNN
+F 4 "GND" H 3350 1700 50  0000 C CNN "2"
+F 5 "Vcc" H 3350 1600 50  0000 C CNN "1"
+	1    3600 1750
 	-1   0    0    1
 $EndComp
@@
 1
 Wire Wire Line
-	5900 2250 5900 2700
-Wire Wire Line
-	4650 2350 4650 2700
+	3800 1750 4650 1750
+Wire Wire Line
+	3800 1650 5900 1650
+$Comp
+L Connector:Conn_01x06_Male J1
+U 1 1 5EF3CD44
+P 3550 4300
+F 0 "J1" H 3350 4350 50  0000 C CNN
+F 1 "Rows" H 3350 4250 50  0000 C CNN
+F 2 "" H 3550 4300 50  0001 C CNN
+F 3 "~" H 3550 4300 50  0001 C CNN
+	1    3550 4300
+	1    0    0    -1
+$EndComp
+Wire Wire Line
+	5900 2900 6050 2900
+Wire Wire Line
+	6000 2800 5900 2800
+$Comp
+L Connector:Conn_01x20_Male J2
+U 1 1 5EF43085
+P 3550 2900
+F 0 "J2" H 3400 2950 50  0000 R CNN
+F 1 "Columns" H 3500 2850 50  0000 R CNN
+F 2 "" H 3550 2900 50  0001 C CNN
+F 3 "~" H 3550 2900 50  0001 C CNN
+	1    3550 2900
+	1    0    0    -1
+$EndComp
+Wire Wire Line
+	6100 3000 5900 3000
+Wire Wire Line
+	6350 3500 5900 3500
+Wire Wire Line
+	6400 3600 5900 3600
+Wire Wire Line
+	6000 2800 6000 2550
+Wire Wire Line
+	6050 2500 6050 2900
+Wire Wire Line
+	6100 3000 6100 2450
+Text Notes 4625 3550 2    31   ~ 0
+Internal\nLED
+Wire Wire Line
+	5900 3100 6150 3100
+Wire Wire Line
+	5900 3200 6200 3200
+Wire Wire Line
+	5900 3300 6250 3300
+Wire Wire Line
+	5900 3400 6300 3400
 $Comp
 L teensy:Teensy++2.0-teensy++20 IC1
 U 1 1 5EB26E81
 P 5300 2450
-F 0 "IC1" H 5275 2465 50  0000 C CNN
-F 1 "Teensy++2.0" H 5275 2374 50  0000 C CNN
+F 0 "IC1" H 5250 1250 50  0000 C CNN
+F 1 "Teensy++2.0" H 5250 1150 50  0000 C CNN
 F 2 "" H 5300 2450 50  0001 C CNN
 F 3 "" H 5300 2450 50  0001 C CNN
@@
 $EndComp
 Wire Wire Line
-	3250 2350 4650 2350
-Wire Wire Line
-	3250 2250 5900 2250
-$Comp
-L Connector:Conn_01x06_Male J1
-U 1 1 5EF3CD44
-P 3000 3000
-F 0 "J1" H 2850 3050 50  0000 C CNN
-F 1 "Rows" H 2850 2950 50  0000 C CNN
-F 2 "" H 3000 3000 50  0001 C CNN
-F 3 "~" H 3000 3000 50  0001 C CNN
-	1    3000 3000
-	1    0    0    -1
-$EndComp
-Wire Wire Line
-	4650 2800 3200 2800
-Wire Wire Line
-	3200 2900 4650 2900
-Wire Wire Line
-	4650 3000 3200 3000
-Wire Wire Line
-	4650 3100 3200 3100
-Wire Wire Line
-	4650 3200 3200 3200
-Wire Wire Line
-	4650 3300 3200 3300
-$Comp
-L Connector:Conn_01x20_Male J2
-U 1 1 5EF43085
-P 3000 4500
-F 0 "J2" H 2750 4550 50  0000 R CNN
-F 1 "Columns" H 2850 4450 50  0000 R CNN
-F 2 "" H 3000 4500 50  0001 C CNN
-F 3 "~" H 3000 4500 50  0001 C CNN
-	1    3000 4500
-	1    0    0    -1
-$EndComp
-Wire Wire Line
-	4650 4500 3200 4500
-Wire Wire Line
-	4650 4400 3200 4400
-Wire Wire Line
-	3200 3600 4650 3600
-Wire Wire Line
-	3200 3700 4650 3700
-Wire Wire Line
-	3200 3800 4650 3800
-Wire Wire Line
-	3200 3900 4650 3900
-Wire Wire Line
-	3200 4000 4650 4000
-Wire Wire Line
-	3200 4100 4650 4100
-Wire Wire Line
-	3200 4200 4650 4200
-Wire Wire Line
-	3200 4300 4650 4300
-Wire Wire Line
-	4650 4600 3200 4600
-Wire Wire Line
-	5950 4750 5950 4600
-Wire Wire Line
-	5950 4600 5900 4600
-Wire Wire Line
-	3200 4800 6050 4800
-Wire Wire Line
-	6050 4800 6050 4500
-Wire Wire Line
-	6050 4500 5900 4500
-Wire Wire Line
-	4600 4750 5950 4750
-Wire Wire Line
-	4600 4700 4600 4750
-Wire Wire Line
-	3200 4700 4600 4700
-Wire Wire Line
-	3200 4900 6150 4900
-Wire Wire Line
-	6150 4900 6150 4400
-Wire Wire Line
-	6150 4400 5900 4400
-Wire Wire Line
-	5900 4300 6250 4300
-Wire Wire Line
-	6250 4300 6250 5000
-Wire Wire Line
-	6250 5000 3200 5000
-Wire Wire Line
-	3200 5100 6350 5100
-Wire Wire Line
-	6350 5100 6350 3600
-Wire Wire Line
-	6350 3600 5900 3600
-Wire Wire Line
-	5900 3500 6450 3500
-Wire Wire Line
-	6450 3500 6450 5200
-Wire Wire Line
-	6450 5200 3200 5200
-Wire Wire Line
-	3200 5300 6550 5300
-Wire Wire Line
-	6550 5300 6550 3000
-Wire Wire Line
-	6550 3000 5900 3000
-Wire Wire Line
-	5900 2900 6650 2900
-Wire Wire Line
-	6650 2900 6650 5400
-Wire Wire Line
-	6650 5400 3200 5400
-Wire Wire Line
-	3200 5500 6750 5500
-Wire Wire Line
-	6750 5500 6750 2800
-Wire Wire Line
-	6750 2800 5900 2800
+	4650 4600 3750 4600
+Wire Wire Line
+	4650 4500 3750 4500
+Wire Wire Line
+	4650 4400 3750 4400
+Wire Wire Line
+	4650 4300 3750 4300
+Wire Wire Line
+	3750 4200 4650 4200
+Wire Wire Line
+	4650 4100 3750 4100
+Wire Wire Line
+	4650 2800 4400 2800
+Wire Wire Line
+	4400 2800 4400 3200
+Wire Wire Line
+	4400 3200 3750 3200
+Wire Wire Line
+	4650 1750 4650 2700
+Wire Wire Line
+	5900 1650 5900 2700
+Wire Wire Line
+	6000 2550 4350 2550
+Wire Wire Line
+	4350 2550 4350 3100
+Wire Wire Line
+	4350 3100 3750 3100
+Wire Wire Line
+	6050 2500 4300 2500
+Wire Wire Line
+	4300 2500 4300 3000
+Wire Wire Line
+	4300 3000 3750 3000
+Wire Wire Line
+	6100 2450 4250 2450
+Wire Wire Line
+	4250 2450 4250 2900
+Wire Wire Line
+	4250 2900 3750 2900
+Wire Wire Line
+	5900 3900 6450 3900
+Wire Wire Line
+	5900 4000 6500 4000
+Wire Wire Line
+	5900 4100 6550 4100
+Wire Wire Line
+	6150 3100 6150 2400
+Wire Wire Line
+	6150 2400 4200 2400
+Wire Wire Line
+	4200 2400 4200 2800
+Wire Wire Line
+	4200 2800 3750 2800
+Wire Wire Line
+	6200 3200 6200 2350
+Wire Wire Line
+	6200 2350 4150 2350
+Wire Wire Line
+	4150 2350 4150 2700
+Wire Wire Line
+	4150 2700 3750 2700
+Wire Wire Line
+	3750 2600 4100 2600
+Wire Wire Line
+	4100 2300 6250 2300
+Wire Wire Line
+	6250 2300 6250 3300
+Wire Wire Line
+	6300 2250 6300 3400
+Wire Wire Line
+	6350 3500 6350 2200
+Wire Wire Line
+	6350 2200 4000 2200
+Wire Wire Line
+	4000 2200 4000 2400
+Wire Wire Line
+	4000 2400 3750 2400
+Wire Wire Line
+	3750 2300 3950 2300
+Wire Wire Line
+	3950 2300 3950 2150
+Wire Wire Line
+	3950 2150 6400 2150
+Wire Wire Line
+	6400 2150 6400 3600
+Wire Wire Line
+	6450 3900 6450 2100
+Wire Wire Line
+	6450 2100 3900 2100
+Wire Wire Line
+	3900 2100 3900 2200
+Wire Wire Line
+	3900 2200 3750 2200
+Wire Wire Line
+	3750 2100 3850 2100
+Wire Wire Line
+	3850 2100 3850 2050
+Wire Wire Line
+	3850 2050 6500 2050
+Wire Wire Line
+	6500 2050 6500 4000
+Wire Wire Line
+	6550 4100 6550 2000
+Wire Wire Line
+	3750 3300 4650 3300
+Wire Wire Line
+	3750 3400 4650 3400
+Wire Wire Line
+	3750 3500 4400 3500
+Wire Wire Line
+	4400 3500 4400 3600
+Wire Wire Line
+	4400 3600 4650 3600
+Wire Wire Line
+	4650 3700 4350 3700
+Wire Wire Line
+	4350 3700 4350 3600
+Wire Wire Line
+	4350 3600 3750 3600
+Wire Wire Line
+	3750 3700 4300 3700
+Wire Wire Line
+	4300 3700 4300 3800
+Wire Wire Line
+	4300 3800 4650 3800
+Wire Wire Line
+	3750 3800 4250 3800
+Wire Wire Line
+	4250 3800 4250 3900
+Wire Wire Line
+	4250 3900 4650 3900
+Wire Wire Line
+	3750 3900 4200 3900
+Wire Wire Line
+	4200 3900 4200 4000
+Wire Wire Line
+	4200 4000 4650 4000
+Wire Wire Line
+	4100 2600 4100 2300
+Wire Wire Line
+	4050 2250 6300 2250
+Wire Wire Line
+	3750 2500 4050 2500
+Wire Wire Line
+	4050 2500 4050 2250
+Wire Wire Line
+	3750 2000 6550 2000
 $EndSCHEMATC

Commit message: Added serial port communication
Both ICs might exchange data through Serial1 port
Parts:
- added J?: Serial IC1, symbol Connector_Generic:Conn_01x02
- renumbered IC1 to IC2
Connections:
- wire segments 88 -> 94
Changed lines of the file:
@@
 L Connector_Generic:Conn_01x02 J1
 U 1 1 5E771D4E
-P 3600 1750
-F 0 "J1" H 3518 1425 50  0001 C CNN
-F 1 "Input 5v" H 3518 1516 50  0000 C CNB
-F 2 "" H 3600 1750 50  0001 C CNN
-F 3 "~" H 3600 1750 50  0001 C CNN
-F 4 "GND" H 3350 1700 50  0000 C CNN "2"
-F 5 "Vcc" H 3350 1600 50  0000 C CNN "1"
-	1    3600 1750
+P 3600 1350
+F 0 "J1" H 3518 1025 50  0001 C CNN
+F 1 "Input 5v" H 3518 1116 50  0000 C CNB
+F 2 "" H 3600 1350 50  0001 C CNN
+F 3 "~" H 3600 1350 50  0001 C CNN
+F 4 "GND" H 3350 1300 50  0000 C CNN "2"
+F 5 "Vcc" H 3350 1200 50  0000 C CNN "1"
+	1    3600 1350
 	-1   0    0    1
 $EndComp
@@
 1
 Wire Wire Line
-	3800 1750 4650 1750
-Wire Wire Line
-	3800 1650 5900 1650
+	3800 1350 4650 1350
+Wire Wire Line
+	3800 1250 5900 1250
 $Comp
 L Connector:Conn_01x06_Male J1
@@
 	5900 3400 6300 3400
 $Comp
-L teensy:Teensy++2.0-teensy++20 IC1
+L teensy:Teensy++2.0-teensy++20 IC2
 U 1 1 5EB26E81
 P 5300 2450
-F 0 "IC1" H 5250 1250 50  0000 C CNN
+F 0 "IC2" H 5250 1250 50  0000 C CNN
 F 1 "Teensy++2.0" H 5250 1150 50  0000 C CNN
 F 2 "" H 5300 2450 50  0001 C CNN
@@
 	4400 3200 3750 3200
 Wire Wire Line
-	4650 1750 4650 2700
-Wire Wire Line
-	5900 1650 5900 2700
+	4650 1350 4650 2700
+Wire Wire Line
+	5900 1250 5900 2700
 Wire Wire Line
 	6000 2550 4350 2550
@@
 Wire Wire Line
 	3750 2000 6550 2000
+$Comp
+L Connector_Generic:Conn_01x02 J?
+U 1 1 5F0A7196
+P 3600 1750
+F 0 "J?" H 3518 1425 50  0001 C CNN
+F 1 "Serial IC1" H 3518 1516 50  0000 C CNB
+F 2 "" H 3600 1750 50  0001 C CNN
+F 3 "~" H 3600 1750 50  0001 C CNN
+F 4 "TX" H 3350 1700 50  0000 C CNN "2"
+F 5 "RX" H 3350 1600 50  0000 C CNN "1"
+	1    3600 1750
+	-1   0    0    1
+$EndComp
+Wire Wire Line
+	4650 3200 4450 3200
+Wire Wire Line
+	4450 3200 4450 1750
+Wire Wire Line
+	4450 1750 3800 1750
+Wire Wire Line
+	3800 1650 4500 1650
+Wire Wire Line
+	4500 1650 4500 3100
+Wire Wire Line
+	4500 3100 4650 3100
 $EndSCHEMATC
