File: electronics/Controller.sch (KiCad schematic (older format))
At the start: 23 parts, among them IC1 Teensy++2.0, J1 Input 5v

Commit message: new backlight schematic (darlington TIP112)
Parts:
- removed Q?: IRF520, Package_TO_SOT_THT:TO-220-3_Vertical, symbol Transistor_FET:IRF540N
- added ...LED.n..., _: LED, symbol Device:LED
- added Q1: TIP112, Package_TO_SOT_THT:TO-220-3_Vertical, symbol Transistor_BJT:TIP120
- added R?: 1K, symbol Device:R
- added R? (x2): 470, symbol Device:R
Connections:
- net GNDREF: now also J?.3 (Pin_3), Q1.3 (E)
- net at J?.1 (Pin_1): now also R?.1
- net at J?.2 (Pin_2): now also R?.1, R?.1
- new net: Q1.1 (B), R?.2
- new net: ...LED.n....1 (K), Q1.2 (C), _.1 (K)
- new net: ...LED.n....2 (A), R?.2
- new net: R?.2, _.2 (A)
Other:
- moved on the sheet: Control, IC1, LCD, Macro, caps, num
